File: wifi-modem.sch (KiCad schematic (older format))
At the start: 46 parts, among them J1 RS232, J2 Power, J3 Speaker, SW1 RESET, SW2 PROG, U1 ESP-12F, U2 MAX3238EAIT, U3 AMS1117-3.3, U4 74HCT541

Commit message: PCB Version 3
Parts:
- added C12, C13, C14: 100nF, Capacitor_SMD:C_0805_2012Metric_Pad1.15x1.40mm_HandSolder, symbol Device:C_Small
- added R17, R18: 1MΩ, Resistor_SMD:R_0805_2012Metric_Pad1.15x1.40mm_HandSolder, symbol Device:R_Small
- added U5: 74LV123, Package_SO:TSSOP-16_4.4x5mm_P0.65mm, symbol 74xx:74HCT123
- U4: footprint Package_SO:SSOP-20_5.3x7.2mm_P0.65mm -> Package_SO:TSSOP-20_4.4x6.5mm_P0.65mm; symbol 74xx:74HCT541 -> wifi-modem-rescue:74HCT541-74xx
Connections:
- net +3V3: now also D1.2 (A), D2.2 (A), D3.2 (A), D4.2 (A), D5.2 (A), D6.2 (A), D7.2 (A), D8.2 (A), C14.2, R17.1, R18.1, U5.11 (Clr), U5.16 (VCC), U5.3 (Clr)
- net GND: now also C14.1, U5.1 (A), U5.8 (GND), U5.9 (A); no longer D1.1 (K), D2.1 (K), D3.1 (K), D4.1 (K), D5.1 (K), D6.1 (K), D7.1 (K), D8.1 (K)
- net at U1.21 (GPIO3/RXD), U2.21 (R1OUT): now also U5.2 (B); no longer U4.8 (A6)
- net at U1.22 (GPIO1/TXD), U2.24 (T1IN): now also U5.10 (B); no longer U4.9 (A7)
- net at R1.2: now also D1.1 (K); no longer D1.2 (A)
- net at R2.2: now also D2.1 (K); no longer D2.2 (A)
- net at R3.2: now also D3.1 (K); no longer D3.2 (A)
- net at R4.2: now also D4.1 (K); no longer D4.2 (A)
- net at R5.2: now also D5.1 (K); no longer D5.2 (A)
- net at R6.2: now also D6.1 (K); no longer D6.2 (A)
- net at R7.2: now also D7.1 (K); no longer D7.2 (A)
- net at R8.2: now also D8.1 (K); no longer D8.2 (A)
- new net: U4.8 (A6), U5.13 (Q)
- new net: U4.9 (A7), U5.5 (Q)
- new net: C13.2, U5.6 (Cext)
- new net: C13.1, R18.2, U5.7 (RCext)
- new net: C12.2, U5.14 (Cext)
- new net: C12.1, R17.2, U5.15 (RCext)
- no-connect marks 27 -> 29
Other:
- moved on the sheet: C1, C10, C11, C2, C3, C4, C5, C6, C7, C8, C9, D1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
